File: tm3130-2481bs.kicad_pcb (KiCad board)
At the start: 2 copper layers, 32.8 x 17.8 mm, 18 parts, among them J1 Conn_01x03_Male, J2 Conn_01x03_Male, U1 TM3130, U2 CA56-12CGKWA

Commit message: Adding manufacturing data
Parts:
- added H3: MountingHole, jlcpcb-tooling:tooling-hole, F.Cu at (126.6, 42.0)
- added H4: MountingHole, jlcpcb-tooling:tooling-hole, F.Cu at (144.0, 42.0)
- added H5: MountingHole, jlcpcb-tooling:tooling-hole, F.Cu at (150.2, 57.0)
Other:
- board size 32.8 x 17.8 mm -> 32.8 x 20 mm
- board text added: "JLCJLCJLCJLC"
